File: AIO-OPAMP/op-amps.kicad_sch (KiCad schematic)
At the start: 30 parts, among them J1 Screw_Terminal_01x02, J10 Conn_01x01_Pin, J11 Conn_01x02, J12 Conn_01x01_Pin, J13 Conn_01x01_Pin, J14 Conn_01x03, J15 Conn_01x03, J16 Conn_01x03, J17 Conn_01x03, J18 Conn_01x02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

Commit message: s
Parts:
- removed J14, J15, J16, J17: Conn_01x03, Connector_PinHeader_2.54mm:PinHeader_1x03_P2.54mm_Vertical, symbol Connector_Generic:Conn_01x03
- removed J18: Conn_01x02, Connector_PinHeader_2.54mm:PinHeader_1x02_P2.54mm_Vertical, symbol Connector_Generic:Conn_01x02
- removed J2: Conn_02x03_Odd_Even, Connector_PinHeader_2.54mm:PinHeader_2x03_P2.54mm_Vertical, symbol Connector_Generic:Conn_02x03_Odd_Even
- removed R1, R2: R, Resistor_THT:R_Axial_DIN0207_L6.3mm_D2.5mm_P7.62mm_Horizontal, symbol Device:R
- added J15: Conn_02x04_Odd_Even, symbol Connector_Generic:Conn_02x04_Odd_Even
- added J2, J20, J21, J22: Conn_01x02, Connector_PinHeader_2.54mm:PinHeader_1x02_P2.54mm_Vertical, symbol Connector_Generic:Conn_01x02
- added RV5: R_Potentiometer, Potentiometer_THT:Potentiometer_Bourns_3296W_Vertical, symbol Device:R_Potentiometer
Connections:
- net GND: now also J11.2 (Pin_2), J9.2 (Pin_2), J15.7 (Pin_7), J2.1 (Pin_1), J20.2 (Pin_2), J21.2 (Pin_2), J22.2 (Pin_2); no longer D1.2 (A), J13.1 (Pin_1)
- net VCC: now also RV5.1
- net VEE: now also D1.2 (A), J13.1 (Pin_1), RV5.3
- net bat+: now also J15.3 (Pin_3)
- net buffer_amp_vo: now also J11.1 (Pin_1)
- net inv_amp_vin: now also J20.1 (Pin_1); no longer J9.1 (Pin_1), J9.2 (Pin_2)
- net inv_amp_vo: now also J21.1 (Pin_1)
- net noninv_amp_vin: now also J9.1 (Pin_1); no longer J11.1 (Pin_1), J11.2 (Pin_2)
- net noninv_amp_vo: now also J22.1 (Pin_1)
- net v_devider: now also J15.5 (Pin_5), RV5.2
- net v_zener: now also J15.1 (Pin_1)
- net at U1.9 (-): now also J15.2 (Pin_2), J15.4 (Pin_4), J15.6 (Pin_6), J15.8 (Pin_8)
- net zero corss renamed cross_detect_out
- net cross_detect_out: now also J2.2 (Pin_2)
Other:
- moved on the sheet: C1, C3, D1, J1, J12, J13, J19, J3, J5, R3, U1B, U1C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

Commit message: in_layout
Parts:
- added J14, J16, J17, J18, J23: Conn_01x01_Pin, Connector_PinHeader_2.54mm:PinHeader_1x01_P2.54mm_Vertical, symbol Connector:Conn_01x01_Pin
Connections:
- net VCC: now also J16.1 (Pin_1)
- net VEE: now also J14.1 (Pin_1)
- net inv_amp_vin: now also J17.1 (Pin_1)
- net at J6.1 (Pin_1), RV3.3, RV4.3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: now also J23.1 (Pin_1)
- net at J10.1 (Pin_1), RV1.2, RV2.1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: now also J18.1 (Pin_1)
Other:
- moved on the sheet: D1, J12, J13, J15, J19, R3, RV5, U1C
