File: AIO-OPAMP/op-amps.kicad_sch (KiCad schematic)
At the start: 34 parts, among them J1 Screw_Terminal_01x02, J10 Conn_01x01_Pin, J11 Conn_01x02, J12 Conn_01x01_Pin, J13 Conn_01x01_Pin, J14 Conn_01x01_Pin, J15 Conn_02x04_Odd_Even, J16 Conn_01x01_Pin, J17 Conn_01x01_Pin, J18 Conn_01x01_Pin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

Commit message: 9
Parts:
- removed C1: C_Polarized, Capacitor_THT:CP_Radial_D8.0mm_P5.00mm, symbol Device:C_Polarized
- added J25, J26: Conn_01x02, Connector_PinHeader_2.54mm:PinHeader_1x02_P2.54mm_input, symbol Connector_Generic:Conn_01x02
- J1: footprint Connector_PinHeader_2.54mm:PinHeader_1x02_P2.54mm_Vertical -> TerminalBlock:TerminalBlock_MaiXu_MX126-5.0-02P_1x02_P5.00mm
- J15: footprint (none) -> Connector_PinHeader_2.54mm:PinHeader_2x04_P2.54mm_Vertical
- J2: footprint Connector_PinHeader_2.54mm:PinHeader_1x02_P2.54mm_Vertical -> Connector_PinHeader_2.54mm:PinHeader_1x02_P2.54mm_input
- J3: footprint TerminalBlock:TerminalBlock_bornier-3_P5.08mm -> TerminalBlock:TerminalBlock_MaiXu_MX126-5.0-03P_1x03_P5.00mm
- RV1, RV2, RV3, RV4, RV5: footprint Potentiometer_THT:Potentiometer_Bourns_3296W_Vertical -> Potentiometer_THT:Potentiometer_ACP_CA9-H5_Horizontal
Connections:
- net GND: now also J25.1 (Pin_1), J25.2 (Pin_2), J26.1 (Pin_1), J26.2 (Pin_2); no longer J2.1 (Pin_1)
- net cross_detect_out: now also J2.1 (Pin_1); no longer J2.2 (Pin_2)
Other:
- moved on the sheet: J2
