File: AIO-OPAMP/op-amps.kicad_pcb (KiCad board)
At the start: 2 copper layers, 31 parts, among them J1 Screw_Terminal_01x02, J10 Conn_01x01_Pin, J11 Conn_01x02, J12 Conn_01x01_Pin, J13 Conn_01x01_Pin, J14 Conn_01x03, J15 Conn_01x03, J16 Conn_01x03, J17 Conn_01x03, J18 Conn_01x02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

Commit message: starting
Parts:
- removed R1, R2: R, Resistor_THT:R_Axial_DIN0207_L6.3mm_D2.5mm_P7.62mm_Horizontal
- added J11: Conn_01x02, Connector_PinHeader_2.54mm:PinHeader_1x02_P2.54mm_Vertical, F.Cu at (224.2, 128.5)
- added J14: Conn_01x01_Pin, Connector_PinHeader_2.54mm:PinHeader_1x01_P2.54mm_Vertical, F.Cu at (210.5, 128.5)
- added J16: Conn_01x01_Pin, Connector_PinHeader_2.54mm:PinHeader_1x01_P2.54mm_Vertical, F.Cu at (210.5, 133.1)
- added J17: Conn_01x01_Pin, Connector_PinHeader_2.54mm:PinHeader_1x01_P2.54mm_Vertical, F.Cu at (210.5, 137.6)
- added J18: Conn_01x01_Pin, Connector_PinHeader_2.54mm:PinHeader_1x01_P2.54mm_Vertical, F.Cu at (210.5, 142.2)
- added J2: Conn_01x02, Connector_PinHeader_2.54mm:PinHeader_1x02_P2.54mm_Vertical, F.Cu at (215.1, 128.5)
- added J20: Conn_01x02, Connector_PinHeader_2.54mm:PinHeader_1x02_P2.54mm_Vertical, F.Cu at (228.8, 128.5)
- added J21: Conn_01x02, Connector_PinHeader_2.54mm:PinHeader_1x02_P2.54mm_Vertical, F.Cu at (233.4, 128.5)
- added J22: Conn_01x02, Connector_PinHeader_2.54mm:PinHeader_1x02_P2.54mm_Vertical, F.Cu at (238.0, 128.5)
- added J23: Conn_01x01_Pin, Connector_PinHeader_2.54mm:PinHeader_1x01_P2.54mm_Vertical, F.Cu at (210.5, 146.8)
- added J9: Conn_01x02, Connector_PinHeader_2.54mm:PinHeader_1x02_P2.54mm_Vertical, F.Cu at (219.6, 128.5)
- added RV5: R_Potentiometer, Potentiometer_THT:Potentiometer_Bourns_3296W_Vertical, F.Cu at (220.8, 136.5)
- J14, J16, J17: value Conn_01x03 -> Conn_01x01_Pin; footprint Connector_PinHeader_2.54mm:PinHeader_1x03_P2.54mm_Vertical -> Connector_PinHeader_2.54mm:PinHeader_1x01_P2.54mm_Vertical
- J15: value Conn_01x03 -> Conn_02x04_Odd_Even
- J18: value Conn_01x02 -> Conn_01x01_Pin; footprint Connector_PinHeader_2.54mm:PinHeader_1x02_P2.54mm_Vertical -> Connector_PinHeader_2.54mm:PinHeader_1x01_P2.54mm_Vertical
- J2: value Conn_02x03_Odd_Even -> Conn_01x02; footprint Connector_PinHeader_2.54mm:PinHeader_2x03_P2.54mm_Vertical -> Connector_PinHeader_2.54mm:PinHeader_1x02_P2.54mm_Vertical
- J20: value Conn_01x04 -> Conn_01x02; footprint Connector_PinHeader_2.54mm:PinHeader_1x06_P2.54mm_Vertical -> Connector_PinHeader_2.54mm:PinHeader_1x02_P2.54mm_Vertical
- J5: footprint Connector_PinHeader_2.54mm:PinHeader_1x02_P2.54mm_input -> Connector_PinHeader_2.54mm:PinHeader_1x02_P2.54mm_Vertical
- moved J20 6.93 mm to (167.0, 98.8)
Connections:
- D1 pad 2: bat- -> VEE
- J11 pad 1: noninv_amp_vin -> buffer_amp_vo
- J11 pad 2: noninv_amp_vin -> bat-
- J13 pad 1: bat- -> VEE
- J14 pad 1: inv_amp_vo -> VEE
- J15 pad 1: noninv_amp_vo -> v_zener
- J15 pad 2: unconnected-(J15-Pin_2-Pad2) -> Net-(J15-Pin_2)
- J15 pad 3: bat- -> bat+
- J16 pad 1: buffer_amp_vo -> VCC
- J17 pad 1: zero corss -> inv_amp_vin
- J18 pad 1: buffer_vin -> Net-(J10-Pin_1)
- J2 pad 1: v_zener -> bat-
- J2 pad 2: Net-(J2-Pin_2) -> cross_detect_out
- J20 pad 1: unconnected-(J20-Pin_1-Pad1) -> inv_amp_vin
- J20 pad 2: unconnected-(J20-Pin_2-Pad2) -> bat-
- J9 pad 1: inv_amp_vin -> noninv_amp_vin
- J9 pad 2: inv_amp_vin -> bat-
- U1 pad 8: zero corss -> cross_detect_out
- U1 pad 9: Net-(J2-Pin_2) -> Net-(J15-Pin_2)
Routing:
- net Net-(J2-Pin_2): track 18.9 -> 0.00 mm
- net Net-(J15-Pin_2): track 0.00 -> 18.9 mm
- net zero corss: track 5.53 -> 0.00 mm
- net cross_detect_out: track 0.00 -> 5.53 mm
- net bat-: track 13.5 -> 12.0 mm
- net VEE: track 7.51 -> 8.98 mm

Commit message: p
Parts:
- removed C1: C_Polarized, Capacitor_THT:CP_Radial_D8.0mm_P5.00mm
- removed the J11 at (234.0, 88.7)
- removed the J11 at (224.2, 128.5)
- removed the J14 at (209.3, 75.0)
- removed the J14 at (210.5, 128.5)
- removed the J16 at (210.5, 133.1)
- removed the J16 at (210.5, 111.5)
- removed the J17 at (210.5, 137.6)
- removed the J17 at (223.5, 112.0)
- removed the J18 at (210.5, 142.2)
- removed the J18 at (234.0, 98.0)
- removed the J2 at (215.1, 128.5)
- removed the J2 at (236.5, 106.6)
- removed the J20 at (167.0, 98.8)
- removed the J20 at (228.8, 128.5)
- removed the J9 at (219.6, 128.5)
- removed the J9 at (197.7, 75.2)
- added J11: Conn_01x02, Connector_PinHeader_2.54mm:PinHeader_1x02_P2.54mm_input, F.Cu at (262.9, 87.7)
- added J14: Conn_01x01_Pin, Connector_PinHeader_2.54mm:PinHeader_1x01_P2.54mm_Vertical, F.Cu at (234.0, 170.9)
- added J16: Conn_01x01_Pin, Connector_PinHeader_2.54mm:PinHeader_1x01_P2.54mm_Vertical, F.Cu at (234.0, 175.5)
- added J17: Conn_01x01_Pin, Connector_PinHeader_2.54mm:PinHeader_1x01_P2.54mm_Vertical, F.Cu at (234.0, 180.1)
- added J18: Conn_01x01_Pin, Connector_PinHeader_2.54mm:PinHeader_1x01_P2.54mm_Vertical, F.Cu at (217.4, 168.7)
- added J2: Conn_01x02, Connector_PinHeader_2.54mm:PinHeader_1x02_P2.54mm_input, F.Cu at (260.5, 96.5)
- added J20: Conn_01x02, Connector_PinHeader_2.54mm:PinHeader_1x02_P2.54mm_input, F.Cu at (164.8, 79.0)
- added J24: Conn_01x02, Connector_PinHeader_2.54mm:PinHeader_1x02_P2.54mm_input, F.Cu at (164.8, 95.0)
- added J25: Conn_01x02, Connector_PinHeader_2.54mm:PinHeader_1x02_P2.54mm_input, F.Cu at (245.0, 80.0)
- added J26: Conn_01x02, Connector_PinHeader_2.54mm:PinHeader_1x02_P2.54mm_input, F.Cu at (178.0, 90.5)
- added J9: Conn_01x02, Connector_PinHeader_2.54mm:PinHeader_1x02_P2.54mm_input, F.Cu at (164.8, 71.0)
- J15: footprint Connector_PinHeader_2.54mm:PinHeader_1x03_P2.54mm_Vertical -> Connector_PinHeader_2.54mm:PinHeader_2x04_P2.54mm_Vertical
- J21, J22, J5: footprint Connector_PinHeader_2.54mm:PinHeader_1x02_P2.54mm_Vertical -> Connector_PinHeader_2.54mm:PinHeader_1x02_P2.54mm_input
- J3: footprint TerminalBlock:TerminalBlock_bornier-3_P5.08mm -> TerminalBlock:TerminalBlock_MaiXu_MX126-5.0-03P_1x03_P5.00mm
- moved J10 108.0 mm to (229.4, 180.1)
- moved J7 96.2 mm to (229.4, 170.9)
- moved J6 91.3 mm to (229.4, 166.3)
- moved J8 90.3 mm to (229.4, 175.5)
- moved J4 79.2 mm to (206.4, 158.7)
- moved J19 72.5 mm to (238.6, 166.3)
- moved J22 64.4 mm to (262.9, 69.0), turned to -90 degrees
- moved C3 60.9 mm to (210.6, 122.5), turned to 0 degrees
- moved J13 60.7 mm to (234.0, 166.3), turned to 0 degrees
- moved J21 58.1 mm to (262.9, 78.3), turned to -90 degrees
- moved J3 53.9 mm to (212.5, 57.0), turned to 180 degrees
- moved R3 49.4 mm to (201.8, 116.5)
- moved D1 47.9 mm to (192.6, 110.5)
- moved J12 46.6 mm to (234.0, 161.7), turned to 0 degrees
- moved J23 37.0 mm to (238.6, 170.9)
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Connections:
- U1 pad 10: buffer_vin -> cross_vin
Routing:
- net bat-: track 12.0 -> 214.0 mm
- net VEE: track 8.98 -> 160.2 mm
- net VCC: track 0.00 -> 142.4 mm
- net buffer_amp_vo: track 3.45 -> 65.8 mm
- net cross_vin: track 0.00 -> 52.0 mm
- net cross_detect_out: track 5.53 -> 53.6 mm
- net noninv_amp_vin: track 15.9 -> 53.6 mm
- net noninv_amp_vo: track 26.4 -> 51.8 mm
- net inv_amp_vo: track 63.0 -> 85.5 mm
- net buffer_amp_vin: track 17.7 -> 40.0 mm
- net buffer_vin: track 15.5 -> 0.00 mm
- net Net-(J23-Pin_1): track 38.9 -> 23.7 mm
- net v_zener: track 15.1 -> 23.9 mm
- net inv_amp_vin: track 7.53 -> 15.1 mm
- net v_devider: track 13.0 -> 20.0 mm
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Other:
- board text removed: "+"
- board text removed: "-"
- board text removed: "Input"
- board text removed: "Inverting"
- board text removed: "Non-Inverting"
- board text removed: "OUT1"
- board text removed: "OUT2"
- board text removed: "OUT3"
- board text removed: "OUT4"
- board text removed: "Zero Level"
- board text removed: "buffer"
