File: AIO-OPAMP/op-amps.kicad_pcb (KiCad board)
At the start: 2 copper layers, 36 parts, among them J1 Screw_Terminal_01x02, J10 Conn_01x01_Pin, J11 Conn_01x02, J12 Conn_01x01_Pin, J13 Conn_01x01_Pin, J14 Conn_01x01_Pin, J15 Conn_02x04_Odd_Even, J16 Conn_01x01_Pin, J17 Conn_01x01_Pin, J18 Conn_01x01_Pin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

Commit message: final_nopins
Parts:
- removed C1: C_Polarized, Capacitor_THT:CP_Radial_D8.0mm_P5.00mm
- removed J10, J12, J13, J14, J16, J17, J18, J6, J7, J8: Conn_01x01_Pin, Connector_PinHeader_2.54mm:PinHeader_1x01_P2.54mm_Vertical
- J1: footprint Connector_PinHeader_2.54mm:PinHeader_1x02_P2.54mm_Vertical -> TerminalBlock:TerminalBlock_MaiXu_MX126-5.0-02P_1x02_P5.00mm
- moved J23 93.0 mm to (218.1, 80.2)
- moved J19 64.4 mm to (224.8, 103.5)
- moved C3 26.4 mm to (185.0, 116.1), turned to 90 degrees
- moved RV5 7.88 mm to (222.4, 111.8), turned to 90 degrees
- moved J4 5.18 mm to (218.2, 71.6)
- moved J25 4.46 mm to (249.4, 80.0)
- moved J1 1.55 mm to (213.5, 111.7), turned to 180 degrees
Routing:
- net bat-: track 216.2 -> 400.6 mm, vias 0 -> 2
- net VCC: track 143.9 -> 250.6 mm
- net VEE: track 160.2 -> 245.7 mm
- net Net-(J10-Pin_1): track 22.1 -> 35.0 mm
- net noninv_amp_vin: track 53.6 -> 56.3 mm
- net inv_amp_vin: track 14.3 -> 13.0 mm
- net v_devider: track 20.0 -> 19.1 mm
- net bat+: track 8.04 -> 8.83 mm
- added copper zone on B.Cu, net bat-
Other:
- board outline added: 134.4 x 70.9 mm
- board text added: "BATT_IN"
- board text added: "J22"
- board text added: "R2"
- board text added: "RF"
- board text added: "R_ZENER"
- board text added: "Ri"
- board text added: "VCC"
- board text added: "VEE"
- board text added: "VOLTGE DEVIDER"
- board text added: "VOLTGE DEVIDER OUT"
- board text added: "ZENER"
- board text added: "buffer intpot"
- board text added: "buffer outpot"
- board text added: "inverting intpot"
- board text added: "inverting outpot"
- board text added: "level detector input"
- board text added: "level detector output"
- board text added: "noninverting intpot"
- board text added: "noninverting outpot"

Commit message: Update op-amps.kicad_pcb
Other:
- board text added: "buffer intput"
- board text added: "inverting intput"
- board text added: "noninverting intput"
- board text removed: "buffer intpot"
- board text removed: "buffer outpot"
- board text removed: "inverting intpot"
- board text removed: "inverting outpot"
- board text removed: "noninverting intpot"
- board text removed: "noninverting outpot"
Changed lines of the file:
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@@
 		)
 	)
-	(gr_text "noninverting\nintpot"
+	(gr_text "noninverting\nintput"
 		(at 152.84 70.68 0)
 		(layer "F.SilkS")
@@
 		)
 	)
-	(gr_text "noninverting\noutpot"
+	(gr_text "noninverting\nintput"
 		(at 272.51 70.11 0)
 		(layer "F.SilkS")
@@
 		)
 	)
-	(gr_text "buffer\noutpot"
+	(gr_text "buffer\nintput"
 		(at 272.57 88.51 0)
 		(layer "F.SilkS")
@@
 		)
 	)
-	(gr_text "inverting\noutpot"
+	(gr_text "inverting\nintput"
 		(at 272.4 79.51 0)
 		(layer "F.SilkS")
@@
 		)
 	)
-	(gr_text "buffer\nintpot"
+	(gr_text "buffer\nintput"
 		(at 152.9 88.08 0)
 		(layer "F.SilkS")
@@
 		)
 	)
-	(gr_text "inverting\nintpot"
+	(gr_text "inverting\nintput"
 		(at 152.73 80.08 0)
 		(layer "F.SilkS")

Commit message: 9
Other:
- board text added: "buffer input"
- board text added: "buffer output"
- board text added: "inverting input"
- board text added: "inverting output"
- board text added: "noninverting input"
- board text added: "noninverting output"
- board text removed: "buffer intput"
- board text removed: "inverting intput"
- board text removed: "noninverting intput"
Changed lines of the file:
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@@
 		)
 	)
-	(gr_text "noninverting\nintput"
+	(gr_text "noninverting\ninput"
 		(at 152.84 70.68 0)
 		(layer "F.SilkS")
@@
 		)
 	)
-	(gr_text "noninverting\nintput"
+	(gr_text "noninverting\noutput"
 		(at 272.51 70.11 0)
 		(layer "F.SilkS")
@@
 		)
 	)
-	(gr_text "buffer\nintput"
+	(gr_text "buffer\noutput"
 		(at 272.57 88.51 0)
 		(layer "F.SilkS")
@@
 		)
 	)
-	(gr_text "inverting\nintput"
+	(gr_text "inverting\noutput"
 		(at 272.4 79.51 0)
 		(layer "F.SilkS")
@@
 		)
 	)
-	(gr_text "buffer\nintput"
+	(gr_text "buffer\ninput"
 		(at 152.9 88.08 0)
 		(layer "F.SilkS")
@@
 		)
 	)
-	(gr_text "inverting\nintput"
+	(gr_text "inverting\ninput"
 		(at 152.73 80.08 0)
 		(layer "F.SilkS")

Commit message: doin
Parts:
- removed J23: Conn_01x01_Pin, Connector_PinHeader_2.54mm:PinHeader_1x01_P2.54mm_Vertical
- R3: moved to B.Cu
- moved R3 0.33 mm to (202.1, 116.6)
