File: AIO-OPAMP/_autosave-op-amps.kicad_pcb (KiCad board)
At the start: 2 copper layers, 36 parts, among them J1 Screw_Terminal_01x02, J10 Conn_01x01_Pin, J11 Conn_01x02, J12 Conn_01x01_Pin, J13 Conn_01x01_Pin, J14 Conn_01x01_Pin, J15 Conn_02x04_Odd_Even, J16 Conn_01x01_Pin, J17 Conn_01x01_Pin, J18 Conn_01x01_Pin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

Commit message: befor flp
Parts:
- moved C1 15.8 mm to (185.2, 101.5)
- moved RV5 7.88 mm to (222.4, 111.8), turned to 90 degrees
Routing:
- net Net-(J10-Pin_1): track 22.1 -> 34.0 mm
- net VEE: track 160.2 -> 170.0 mm
- net v_devider: track 20.0 -> 15.7 mm
- net VCC: track 143.9 -> 140.8 mm
- net noninv_amp_vin: track 53.6 -> 55.6 mm
Changed lines of the file:
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@@
 	(footprint "Potentiometer_THT:Potentiometer_ACP_CA9-H5_Horizontal"
 		(layer "F.Cu")
-		(at 230.17 110.495)
+		(at 222.4 111.78 90)
 		(descr "Potentiometer, horizontal, ACP CA9-H5, http://www.acptechnologies.com/wp-content/uploads/2017/05/02-ACP-CA9-CE9.pdf")
 		(tags "Potentiometer horizontal ACP CA9-H5")
 		(property "Reference" "RV5"
-			(at 0 -3.65 0)
+			(at 0 -3.65 90)
 			(layer "F.SilkS")
 			(effects
@@
 		)
 		(property "Value" "R_Potentiometer"
-			(at 0 8.65 0)
+			(at 0 8.65 90)
 			(layer "F.Fab")
 			(effects
@@
 		)
 		(property "Datasheet" "~"
-			(at 0 0 0)
+			(at 0 0 90)
 			(layer "F.Fab")
 			(hide yes)
@@
 		)
 		(property "Description" "Potentiometer"
-			(at 0 0 0)
+			(at 0 0 90)
 			(layer "F.Fab")
 			(hide yes)
@@
 		(attr through_hole)
 		(fp_line
-			(start -0.11 -2.51)
-			(end 4.91 -2.51)
-			(stroke
-				(width 0.12)
-				(type solid)
-			)
-			(layer "F.SilkS")
-		)
-		(fp_line
-			(start -0.11 -1.396)
-			(end -0.11 -2.51)
+			(start 4.91 -2.51)
+			(end 4.91 1.103)
 			(stroke
 				(width 0.12)
@@
 		)
 		(fp_line
-			(start -0.11 3.604)
-			(end -0.11 1.396)
+			(start -0.11 -2.51)
+			(end 4.91 -2.51)
 			(stroke
 				(width 0.12)
@@
 		)
 		(fp_line
-			(start -0.11 3.604)
-			(end -0.11 1.396)
+			(start -0.11 -1.396)
+			(end -0.11 -2.51)
 			(stroke
 				(width 0.12)
@@
 		)
 		(fp_line
-			(start -0.11 7.51)
-			(end -0.11 6.396)
+			(start 4.91 0.89)
+			(end 4.91 1.103)
 			(stroke
 				(width 0.12)
@@
 		)
 		(fp_line
-			(start 4.91 -2.51)
-			(end 4.91 1.103)
+			(start -0.11 3.604)
+			(end -0.11 1.396)
 			(stroke
 				(width 0.12)
@@
 		)
 		(fp_line
-			(start 4.91 0.89)
-			(end 4.91 1.103)
+			(start -0.11 3.604)
+			(end -0.11 1.396)
 			(stroke
 				(width 0.12)
@@
 			(layer "F.SilkS")
 		)
+		(fp_line
+			(start -0.11 7.51)
+			(end -0.11 6.396)
+			(stroke
+				(width 0.12)
+				(type solid)
+			)
+			(layer "F.SilkS")
+		)
 		(fp_rect
 			(start -1.42 -2.66)
@@
 		)
 		(fp_text user "${REFERENCE}"
-			(at 2.4 2.5 0)
+			(at 2.4 2.5 90)
 			(layer "F.Fab")
 			(effects
@@
 		)
 		(pad "1" thru_hole circle
-			(at 0 0)
+			(at 0 0 90)
 			(size 2.34 2.34)
 			(drill 1.3)
@@
 		)
 		(pad "2" thru_hole circle
-			(at 5 2.5)
+			(at 5 2.5 90)
 			(size 2.34 2.34)
 			(drill 1.3)
@@
 		)
 		(pad "3" thru_hole circle
-			(at 0 5)
+			(at 0 5 90)
 			(size 2.34 2.34)
 			(drill 1.3)
@@
 	(footprint "Capacitor_THT:CP_Radial_D8.0mm_P5.00mm"
 		(layer "F.Cu")
-		(at 171.14 108.65)
+		(at 185.24 101.54)
 		(descr "CP, Radial series, Radial, pin pitch=5.00mm, diameter=8mm, height=16mm, Electrolytic Capacitor")
 		(tags "CP Radial series Radial pin pitch 5.00mm diameter 8mm height 16mm Electrolytic Capacitor")
@@
 	)
 	(segment
-		(start 210.597349 123.587349)
-		(end 210.597349 122.5)
-		(width 0.5)
-		(layer "B.Cu")
-		(net 1)
-	)
-	(segment
-		(start 211.51 125)
-		(end 211.51 124.5)
-		(width 0.5)
-		(layer "B.Cu")
-		(net 1)
-	)
-	(segment
 		(start 201.81 116.5)
 		(end 204.597349 116.5)
@@
 	)
 	(segment
-		(start 215.665 125)
-		(end 211.51 125)
+		(start 210.57 125)
+		(end 210.57 122.527349)
 		(width 0.5)
 		(layer "B.Cu")
@@
 	)
 	(segment
-		(start 204.597349 116.5)
+		(start 210.57 122.527349)
 		(end 210.597349 122.5)
 		(width 0.5)
@@
 	)
 	(segment
-		(start 211.51 124.5)
-		(end 210.597349 123.587349)
+		(start 217.18 125)
+		(end 210.57 125)
 		(width 0.5)
 		(layer "B.Cu")
@@
 	)
 	(segment
-		(start 179.71 81.33)
-		(end 182.3 83.92)
+		(start 204.597349 116.5)
+		(end 210.597349 122.5)
 		(width 0.5)
 		(layer "B.Cu")
@@
 	)
 	(segment
-		(start 162.5 75)
-		(end 179.5 75)
+		(start 222.4 111.78)
+		(end 222.4 119.78)
 		(width 0.5)
 		(layer "B.Cu")
@@
 	)
 	(segment
-		(start 230.17 110.495)
-		(end 215.665 125)
+		(start 179.71 81.33)
+		(end 182.3 83.92)
+		(width 0.5)
+		(layer "B.Cu")
+		(net 1)
+	)
+	(segment
+		(start 162.5 75)
+		(end 179.5 75)
 		(width 0.5)
 		(layer "B.Cu")
@@
 	)
 	(segment
-		(start 215.7975 119.7875)
-		(end 225.09 110.495)
+		(start 222.4 119.78)
+		(end 217.18 125)
 		(width 0.5)
 		(layer "B.Cu")
-		(net 2)
+		(net 1)
 	)
 	(segment
@@
 	)
 	(segment
-		(start 212.5 57)
-		(end 220.5 65)
+		(start 220.27 109.45)
+		(end 215.597349 114.122651)
 		(width 0.5)
 		(layer "B.Cu")
@@
 	)
 	(segment
-		(start 220.5 65)
-		(end 264 65)
+		(start 215.597349 119.587349)
+		(end 215.597349 122.5)
 		(width 0.5)
 		(layer "B.Cu")
@@
 	)
 	(segment
-		(start 263.08 83.92)
-		(end 211.5 83.92)
+		(start 212.5 57)
+		(end 220.5 65)
 		(width 0.5)
 		(layer "B.Cu")
@@
 	)
 	(segment
-		(start 215.597349 119.987651)
-		(end 215.7975 119.7875)
+		(start 227.4 111.78)
+		(end 225.07 109.45)
 		(width 0.5)
 		(layer "B.Cu")
@@
 	)
 	(segment
+		(start 220.5 65)
+		(end 264 65)
+		(width 0.5)
+		(layer "B.Cu")
+		(net 2)
+	)
+	(segment
+		(start 263.08 83.92)
+		(end 211.5 83.92)
+		(width 0.5)
+		(layer "B.Cu")
+		(net 2)
+	)
+	(segment
+		(start 206.51 110.5)
+		(end 215.597349 119.587349)
+		(width 0.5)
+		(layer "B.Cu")
+		(net 2)
+	)
+	(segment
 		(start 266 67)
 		(end 266 81)
@@
 	)
 	(segment
-		(start 264 65)
-		(end 266 67)
+		(start 225.07 109.45)
+		(end 220.27 109.45)
 		(width 0.5)
 		(layer "B.Cu")
@@
 	)
 	(segment
-		(start 215.597349 122.5)
-		(end 215.597349 119.987651)
+		(start 264 65)
+		(end 266 67)
 		(width 0.5)
 		(layer "B.Cu")
@@
 	)
 	(segment
-		(start 206.51 110.5)
-		(end 215.7975 119.7875)
+		(start 215.597349 114.122651)
+		(end 215.597349 122.5)
 		(width 0.5)
 		(layer "B.Cu")
@@
 	)
 	(segment
-		(start 212.51 106.5)
-		(end 212 105.99)
+		(start 224.9 106.78)
+		(end 224.62 106.5)
 		(width 0.5)
 		(layer "B.Cu")
@@
 	)
 	(segment
-		(start 212 105.99)
-		(end 212 103.5)
+		(start 224.62 106.5)
+		(end 212.51 106.5)
 		(width 0.5)
 		(layer "B.Cu")
@@
 	)
 	(segment
-		(start 227.63 110.495)
-		(end 223.635 106.5)
+		(start 212 105.99)
+		(end 212 103.5)
 		(width 0.5)
 		(layer "B.Cu")
@@
 	)
 	(segment
-		(start 223.635 106.5)
-		(end 212.51 106.5)
+		(start 212.51 106.5)
+		(end 212 105.99)
 		(width 0.5)
 		(layer "B.Cu")
@@
 	(segment
 		(start 186.69 80.35)
-		(end 182.4 80.35)
+		(end 185.9 80.35)
 		(width 0.8)
 		(layer "B.Cu")
@@
 	)
 	(segment
+		(start 192 71)
+		(end 185.9 77.1)
+		(width 0.5)
+		(layer "B.Cu")
+		(net 9)
+	)
+	(segment
 		(start 187.28 80.36)
 		(end 186.7 80.36)
@@
 	)
 	(segment
+		(start 185.9 80.35)
+		(end 182.4 80.35)
+		(width 0.8)
+		(layer "B.Cu")
+		(net 9)
+	)
+	(segment
+		(start 185.9 77.1)
+		(end 185.9 80.35)
+		(width 0.5)
+		(layer "B.Cu")
+		(net 9)
+	)
+	(segment
 		(start 188.8 78.84)
 		(end 187.28 80.36)
@@
 	)
 	(segment
-		(start 204 71)
+		(start 209.88 81.38)
+		(end 208.5 80)
+		(width 0.8)
+		(layer "B.Cu")
+		(net 17)
+	)
+	(segment
+		(start 208.5 78)
+		(end 207 76.5)
+		(width 0.8)
+		(layer "B.Cu")
+		(net 17)
+	)
+	(segment
+		(start 167.29 68.56)
 		(end 164.85 71)
 		(width 0.8)
@@
 	)
 	(segment
-		(start 207 74)
-		(end 204 71)
+		(start 201.56 68.56)
+		(end 167.29 68.56)
 		(width 0.8)
 		(layer "B.Cu")
@@
 	)
 	(segment
-		(start 208.5 78)
-		(end 207 76.5)
+		(start 207 74)
+		(end 201.56 68.56)
 		(width 0.8)
 		(layer "B.Cu")
@@
 		(width 0.8)
 		(layer "B.Cu")
-		(net 17)
-	)
-	(segment
-		(start 209.88 81.38)
-		(end 208.5 80)
-		(width 0.8)
-		(layer "B.Cu")
